File: ece16.kicad_sch (KiCad schematic)
At the start: 55 parts, among them U1 LP5907MFX-3.3, U2 ESP32-S3-MINI-1-N8, U3 ADXL335, U4 DM-OLED096-636, U5 LP5907MFX-1.8, U6 MAX30101EFD_T

Commit message: Updated schematic Accomplished --------- N/A
In Progress
---------
N/A

Errors
----------
N/A

Next
----------
N/A
Parts:
- removed C9: 0.1uF, Capacitor_SMD:C_0402_1005Metric, symbol Device:C
- removed SW1: ~, customFootprints:rockerSwitch-434133025816, symbol custom:Tactile_Switch
- added D3, D6, D7: LED, symbol Device:LED
- added J1: Conn_01x06_Socket, Connector_PinHeader_2.54mm:PinHeader_1x06_P2.54mm_Horizontal, symbol Connector:Conn_01x06_Socket
- added R10, R11, R12, R16, R18, R19: 1k, symbol Device:R_US
- added R20: 10k, Resistor_SMD:R_0402_1005Metric, symbol Device:R_US
- added SW1, SW3, SW4, SW5: ~, customFootprints:rockerSwitch-434133025816, symbol custom:rockerSwitch
Connections:
- net +1.8V: now also J1.6 (Pin_6)
- net +3V3: now also J1.2 (Pin_2), R19.1
- net Boot: now also SW1.1
- net EN: now also R20.2; no longer C4.2, SW2.1
- net GND: now also D3.1 (K), D6.1 (K), D7.1 (K), J1.1 (Pin_1), R11.1, R12.1, R16.1, SW1.2, SW3.2, SW4.2, SW5.2
- net SCL: now also J1.4 (Pin_4)
- net SDA: now also J1.3 (Pin_3)
- net U-LED1: now reaches U2.19 (IO15)
- net U-LED1: now also R10.1
- net U-LED2: now reaches U2.20 (IO16)
- net U-LED2: now also R18.1
- new net: D6.2 (A), R18.2
- new net: D3.2 (A), R10.2
- new net: C4.2, R20.1, SW2.1
- new net: D7.2 (A), R19.2
- new net UB1: R12.2, SW3.1
- new net UB2: R11.2, SW4.1
- new net UB3: R16.2, SW5.1
- no-connect marks 47 -> 45
Other:
- note added: "User Button 1"
- note added: "User Button 2"
- note added: "User Button 3"
- moved on the sheet: BT1, C12, C13, C14, C15, C19, C20, C21, D4, R13, R14, R3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

Commit message: Before you delete and reset everything
Parts:
- removed C1, C2, C7, C8: 0.1uF, Capacitor_SMD:C_0402_1005Metric, symbol Device:C_Small
- removed R12, R16: 1k, symbol Device:R_US
- removed TP1: TestPoint, TestPoint:TestPoint_Keystone_5000-5004_Miniature, symbol Connector:TestPoint
- removed U3: ADXL335, ADXL335:LFCSP-16, symbol ADXL335:ADXL335
- added C1, C2: 0.1uF, Capacitor_SMD:C_0402_1005Metric, symbol Device:C
- added J2: Conn_01x03_Pin, Connector_PinHeader_2.54mm:PinHeader_1x03_P2.54mm_Vertical, symbol Connector:Conn_01x03_Pin
- added U3: LSM6DSOXTR, LSM6DSOXTR:PQFN50P250X300X86-14N, symbol LSM6DSOXTR:LSM6DSOXTR
- BT1: MANUFACTURER 485-1769 -> PRT-09749
- D3, D6, D7: footprint (none) -> LED_SMD:LED_0603_1608Metric; MANUFACTURER (none) -> APHHS1005SURCK
- D4: MANUFACTURER LTST-S270KRKT -> APHHS1005SURCK
- J1: footprint Connector_PinHeader_2.54mm:PinHeader_1x06_P2.54mm_Horizontal -> Connector_PinHeader_2.54mm:PinHeader_1x06_P2.54mm_Vertical
- R10, R18, R19: value 1k -> 510; footprint (none) -> Resistor_SMD:R_0402_1005Metric; MANUFACTURER (none) -> ERJ-2BQJR51X
- R11: footprint (none) -> Resistor_SMD:R_0402_1005Metric; MANUFACTURER (none) -> ERA-2AED512X
Connections:
- net +3V3: now also R11.2, C1.1, C2.1, J2.1 (Pin_1), U3.5 (VDDIO), U3.8 (VDD)
- net +5V: now also C19.1, D4.2 (A), MCP73831T1.4 (VDD)
- net GND: now also C1.2, C2.2, J2.3 (Pin_3), U3.1 (SDO/SA0), U3.2 (SDX), U3.3 (SCX), U3.6 (GND), U3.7 (GND); no longer R11.1
- net SCL: now also U2.28 (IO33), U3.13 (SCL); no longer U2.13 (IO9)
- net SDA: now also U2.29 (IO34), U3.14 (SDA); no longer U2.12 (IO8)
- net UB1: now also U2.31 (IO35)
- net UB2: now also U2.32 (IO36); no longer R11.2
- net UB3: now also U2.33 (IO37)
- net T1: now reaches U2.21 (IO17)
- net T1: now also J2.2 (Pin_2)
- net STAT: no longer names the net of MCP73831T1.1 (STAT), R13.2
- new net: R11.1, U3.12 (CS)
- new net INT1: U3.4 (INT1)
- new net INT2: U3.9 (INT2)
- no-connect marks 45 -> 37
Other:
- note removed: "Check Batt, GND & OLED insertion direction"
- moved on the sheet: BT1, C10, C11, C12, C13, C14, C15, C16, C17, C18, C19, C5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
